Commit message: Untill collisions

File: p_group8_description/urdf/p_randomName.gazebo.xacro (robot description, xacro)
@@ -4,7 +4,21 @@
   <xacro:arg name="camera_visual" default="false"/>
   <xacro:arg name="imu_visual"    default="false"/>
+  <xacro:arg name="player_color" default="Orange" /> <!-- e.g. Red, Orange. Must exist in Gazebo/Colors and be defined in properties.xacro.-->
   <gazebo reference="base_link">
+<!--    Collision sensor-->
+    <sensor name="base_link" type="contact">
+      <update_rate>1000.0</update_rate>
+      <always_on>true</always_on>
+      <contact>
+        <collision> "base_footprint_fixed_joint_lump__base_link_collision" </collision>
+      </contact>
+      <plugin name="base_link_contact_sensor_plugin" filename="libgazebo_ros_bumper.so">
+        <bumperTopicName>contact</bumperTopicName>
+        <frameName>world</frameName>
+      </plugin>
+    </sensor>
+<!--    Color of robot-->
 <!--    <material>Gazebo/Yellow</material>-->
-<!--    <material>Gazebo/${player_color}</material>-->
+    <material>Gazebo/${player_color}</material>
   </gazebo>
   <gazebo reference="wheel_left_link">

Commit message: -Multiple robot environment creation -Loading parameters from YAML file -Team configuration DONE
Next steps:
-Collisions

File: p_group8_description/urdf/p_randomName.gazebo.xacro (robot description, xacro)
@@ -4,12 +4,12 @@
   <xacro:arg name="camera_visual" default="false"/>
   <xacro:arg name="imu_visual"    default="false"/>
-  <xacro:arg name="player_color" default="Orange" /> <!-- e.g. Red, Orange. Must exist in Gazebo/Colors and be defined in properties.xacro.-->
+  <xacro:arg name="player_color" default="Orange" />
   <gazebo reference="base_link">
-<!--    Collision sensor-->
+  <!--    Collision sensor-->
     <sensor name="base_link" type="contact">
       <update_rate>1000.0</update_rate>
       <always_on>true</always_on>
       <contact>
-        <collision> "base_footprint_fixed_joint_lump__base_link_collision" </collision>
+        <collision> "base_footprint_fixed_joint_lump__base_link_collision_2" </collision>
       </contact>
       <plugin name="base_link_contact_sensor_plugin" filename="libgazebo_ros_bumper.so">
@@ -18,6 +18,4 @@
       </plugin>
     </sensor>
-<!--    Color of robot-->
-<!--    <material>Gazebo/Yellow</material>-->
     <material>Gazebo/${player_color}</material>
   </gazebo>
@@ -149,5 +147,4 @@
     </sensor>
   </gazebo>
-<!--link : https://www.raspberrypi.org/documentation/hardware/camera/-->
   <gazebo reference="camera_rgb_frame">
     <sensor type="camera" name="Pi Camera">

File: p_group8_description/urdf/p_randomName.urdf.xacro (robot description, xacro)
@@ -1,14 +1,14 @@
 <?xml version="1.0" ?>
 <robot name="team_hunt_player" xmlns:xacro="http://ros.org/wiki/xacro">
-<!--  Arguments - arguments are used as: $(arg argument) -->
+  <!--  Arguments - arguments are used as: $(arg argument) -->
   <xacro:arg name="player_name"  default="p_randomName"/>
   <xacro:arg name="player_color"  default="Red"/>
-<!-- Copying arguments to properties so that they are visible in the included xacros - properties are used as ${property} -->
+  <!-- Copying arguments to properties so that they are visible in the included xacros - properties are used as ${property} -->
   <xacro:property name="player_name" value="$(arg player_name)"/>
   <xacro:property name="player_color" value="$(arg player_color)"/>
-<!-- Including other xacro files -->
+  <!-- Including other xacro files -->
   <xacro:include filename="$(find p_group8_description)/urdf/properties.xacro"/>
   <xacro:include filename="$(find p_group8_description)/urdf/p_randomName.gazebo.xacro"/>
-<!-- Defining links and joints -->
+  <!-- Defining links and joints -->
   <link name="base_footprint"/>
   <joint name="base_joint" type="fixed">
@@ -23,14 +23,4 @@
         <mesh filename="package://turtlebot3_description/meshes/bases/waffle_pi_base.stl" scale="0.001 0.001 0.001"/>
       </geometry>
-      <!--
-      DEFINING THE MATERIAL:
-        <material> (optional)
-          The material of the visual element.
-        <color> (optional)
-          rgba The color of a material specified by set of four numbers representing red/green/blue/alpha, each in the range of [0,1].
-        <texture> (optional)
-          The texture of a material is specified by a filename
-      See: http://wiki.ros.org/urdf/XML/link chapter 3
-      -->
       <material name="$(arg player_color)"/>
     </visual>

File: p_group8_description/urdf/player.gazebo.urdf.macro.xacro (robot description, xacro)
@@ -26,6 +26,5 @@
     <maxVel>0.1</maxVel>
     <fdir1>1 0 0</fdir1>
-    <!-- Gazebo properties are global: https://answers.ros.org/question/216975/loading-variables-with-xacroinclude/ -->
-<!--    <material>Gazebo/${player_color}</material>-->
+  <!-- Gazebo properties are global: https://answers.ros.org/question/216975/loading-variables-with-xacroinclude/ -->
   </gazebo>
   <gazebo reference="wheel_right_link">
@@ -37,6 +36,4 @@
     <maxVel>0.01</maxVel>
     <fdir1>1 0 0</fdir1>
-    <!-- Gazebo properties are global: https://answers.ros.org/question/216975/loading-variables-with-xacroinclude/ -->
-<!--    <material>Gazebo/${player_color}</material>-->
   </gazebo>
   <gazebo reference="caster_back_right_link">
@@ -66,6 +63,6 @@
   </gazebo>
   <!--Using gazebo or ROS native controller for differential drives -->
-  <!-- TODO: Understand the next line of code: -->
-  <xacro:include filename="$(find p_group8_description)/urdf/ros_diff_drive.gazebo.xacro"/>
+<!--   TODO: Understand the next line of code: -->
+<!--  <xacro:include filename="$(find p_group8_description)/urdf/ros_diff_drive.gazebo.xacro"/>-->
 <!--  Using ROS diff drive controller ... much slower-->
 <!--  <xacro:include filename="$(find p_moliveira_description)/urdf/ros_control.gazebo.xacro"/>-->

File: p_group8_description/urdf/properties.xacro (robot description, xacro)
@@ -3,14 +3,5 @@
     <!--Read common properties from turtlebot3 and then add missing stuff -->
     <xacro:include filename="$(find turtlebot3_description)/urdf/common_properties.xacro"/>
-    <material name="Yellow">
-        <color rgba="1.0 1.0 0.0 1.0"/>
-    </material>
-    <material name="Orange">
-        <color rgba="1.0 0.4 0.0 1.0"/>
-    </material>
-<!--    <material name="sarascolor">-->
-<!--        <color rgba="0.2 0.5 0.8 1.0"/>-->
-<!--    </material>-->
-    <!-- Team hunt player colors-->
+    <!-- TeamHunt player colors -->
     <material name="Red">
     <color rgba="1.0 0.0 0.0 1.0"/>
@@ -22,3 +13,11 @@
     <color rgba="0.0 0.0 1.0 1.0"/>
     </material>
+    <!-- TODO: See if useful -->
+    <!-- TeamHunt 'Joker' player colors -->
+    <material name="Yellow">
+        <color rgba="1.0 1.0 0.0 1.0"/>
+    </material>
+    <material name="Orange">
+        <color rgba="1.0 0.4 0.0 1.0"/>
+    </material>
 </robot>

Commit message: -Multiple robot environment creation -Loading parameters from YAML file -Team configuration -Collisions DONE
Next step:
-Arena mapping

File: p_group8_description/urdf/p_randomName.gazebo.xacro (robot description, xacro)
@@ -11,5 +11,5 @@
       <always_on>true</always_on>
       <contact>
-        <collision> "base_footprint_fixed_joint_lump__base_link_collision_2" </collision>
+        <collision>base_footprint_fixed_joint_lump__base_link_collision</collision>
       </contact>
       <plugin name="base_link_contact_sensor_plugin" filename="libgazebo_ros_bumper.so">
